File: athena_board.sch (KiCad schematic (older format))
At the start: 44 parts, among them IC1 ATMEGA1284P-A, J1 U Motor, J10 HEATER1, J11 U_limit, J12 HEATER2, J15 V_limit, J16 W_limit, J2 V Motor, J3 Expansion, J4 W Motor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

Commit message: Added one Ideal capacitor, removed 3.3V
Parts:
- removed C3: 100uF, Capacitor_SMD:C_1206_3216Metric_Pad1.42x1.75mm_HandSolder, symbol athena_board-rescue:CP-athena-cache
- removed C4: 10uF, Capacitor_SMD:C_1206_3216Metric_Pad1.42x1.75mm_HandSolder, symbol athena_board-rescue:C-athena-cache
- removed U1: AZ2940T-3.3E1, Package_TO_SOT_THT:TO-220-3_Vertical, symbol Regulator_Linear:MCP1826S
- added C?: 22uF @ 50V, symbol athena_board-rescue:CP-athena-cache
- A1, A2, A3, A4: symbol Driver_Motor:Pololu_Breakout_A4988 -> athena_board-rescue:Pololu_Breakout_A4988-Driver_Motor
- J1, J10, J12, J2, J4, J5: symbol Connector:Screw_Terminal_01x04 -> athena_board-rescue:Screw_Terminal_01x04-Connector
- J11, J15, J16, J8, J9: symbol Connector:Screw_Terminal_01x02 -> athena_board-rescue:Screw_Terminal_01x02-Connector
- J3: symbol Connector_Generic:Conn_02x09_Counter_Clockwise -> athena_board-rescue:Conn_02x09_Counter_Clockwise-Connector_Generic
- J7: symbol Connector:Barrel_Jack_MountingPin -> athena_board-rescue:Barrel_Jack_MountingPin-Connector
- P1: symbol Connector_Generic:Conn_01x04 -> athena_board-rescue:Conn_01x04-Connector_Generic
- P2: symbol Connector_Generic:Conn_01x13 -> athena_board-rescue:Conn_01x13-Connector_Generic
- P3: symbol Connector_Generic:Conn_02x13_Odd_Even -> athena_board-rescue:Conn_02x13_Odd_Even-Connector_Generic
- Y1: symbol Device:Crystal -> athena_board-rescue:Crystal-Device
Connections:
- net labels added: +5V-power
- net labels removed: +3.3V, +5V
Other:
- note added: "Need to use Stagard THT footprint to fit boards."
- moved on the sheet: C7
